Commit message: fixed the bug-No valid hardware interface element found in joint

File: agvs_description/urdf/agvs.urdf.xacro (robot description, xacro)
@@ -114,5 +114,7 @@
   <transmission name="joint_bmw_trans">
 	 <type>transmission_interface/SimpleTransmission</type>
-     <joint name="joint_back_motor_wheel" />
+     <joint name="joint_back_motor_wheel" >
+      	    <hardwareInterface>hardware_interface/EffortJointInterface</hardwareInterface>
+     </joint>
      <actuator name="joint_bmw_motor">
 	    <hardwareInterface>EffortJointInterface</hardwareInterface>
@@ -153,5 +155,7 @@
   <transmission name="joint_bw_trans">
 	 <type>transmission_interface/SimpleTransmission</type>
-     <joint name="joint_back_wheel" />
+     <joint name="joint_back_wheel" >
+      <hardwareInterface>hardware_interface/EffortJointInterface</hardwareInterface>
+    </joint>
      <actuator name="joint_bw_motor">
 	   <!-- hardwareInterface>EffortJointInterface</hardwareInterface -->
@@ -193,5 +197,7 @@
   <transmission name="joint_fmw_trans">
 	 <type>transmission_interface/SimpleTransmission</type>
-     <joint name="joint_front_motor_wheel" />
+     <joint name="joint_front_motor_wheel" >
+      <hardwareInterface>hardware_interface/EffortJointInterface</hardwareInterface>
+    </joint>
      <actuator name="joint_fmw_motor">
 	   <hardwareInterface>EffortJointInterface</hardwareInterface>
@@ -233,5 +239,7 @@
   <transmission name="joint_fw_trans">
 	 <type>transmission_interface/SimpleTransmission</type>
-     <joint name="joint_front_wheel" />
+     <joint name="joint_front_wheel" >
+      <hardwareInterface>hardware_interface/EffortJointInterface</hardwareInterface>
+    </joint>
      <actuator name="joint_fw_motor">
 	   <!-- hardwareInterface>EffortJointInterface</hardwareInterface -->
@@ -273,5 +281,7 @@
   <transmission name="joint_swl_trans">
 	 <type>transmission_interface/SimpleTransmission</type>
-     <joint name="joint_side_wheel_left" />
+     <joint name="joint_side_wheel_left" >
+      <hardwareInterface>hardware_interface/EffortJointInterface</hardwareInterface>
+    </joint>
      <actuator name="joint_swl_motor">
 	   <hardwareInterface>EffortJointInterface</hardwareInterface>
@@ -312,5 +322,7 @@
   <transmission name="joint_swr_trans">
 	 <type>transmission_interface/SimpleTransmission</type>
-     <joint name="joint_side_wheel_right" />
+     <joint name="joint_side_wheel_right" >
+      <hardwareInterface>hardware_interface/EffortJointInterface</hardwareInterface>
+    </joint>
      <actuator name="joint_swr_motor">
 	   <hardwareInterface>EffortJointInterface</hardwareInterface>
@@ -347,5 +359,7 @@
   <transmission name="joint_elevator_trans">
 	 <type>transmission_interface/SimpleTransmission</type>
-     <joint name="elevator_joint" />
+     <joint name="elevator_joint" >
+      <hardwareInterface>hardware_interface/EffortJointInterface</hardwareInterface>
+    </joint>
      <actuator name="elevator_motor">
 		<hardwareInterface>EffortJointInterface</hardwareInterface>
